File: debug-board/kicad/field_programmable_smartwatch.sch (KiCad schematic (older format))
At the start: 41 parts, among them IC1 BQ24040DSQR, IC2 STM32WB55CEU6, J1 SPI_Header, J2 LPUART_Header, J3 DX07S016JA1R1500, J4 GPIO_Header, Q1 Q_PMOS_DGS, SW2 SW_DIP_x01, Y1 32M, Y2 32.768k

Commit message: Reworking debug board design
Parts:
- removed J1: SPI_Header, Connector_PinSocket_2.54mm:PinSocket_1x04_P2.54mm_Vertical, symbol Connector:Conn_01x04_Male
- removed J2: LPUART_Header, Connector_PinHeader_2.54mm:PinHeader_1x02_P2.54mm_Vertical, symbol Connector:Conn_01x02_Male
- removed J4: GPIO_Header, Connector_PinHeader_2.54mm:PinHeader_1x09_P2.54mm_Vertical, symbol Connector:Conn_01x09_Male
- removed SW2: SW_DIP_x01, Button_Switch_SMD:SW_DIP_SPSTx01_Slide_6.7x4.1mm_W6.73mm_P2.54mm_LowProfile_JPin, symbol Switch:SW_DIP_x01
- added J1: Conn_01x16_Male, Connector_PinHeader_2.54mm:PinHeader_1x16_P2.54mm_Vertical, symbol Connector:Conn_01x16_Male
- added J2: Conn_01x12_Male, Connector_PinHeader_2.54mm:PinHeader_1x12_P2.54mm_Vertical, symbol Connector:Conn_01x12_Male
- added R4: 100k, Resistor_SMD:R_0402_1005Metric, symbol Device:R_Small
- added SW1, SW2: SW_Push, Button_Switch_SMD:SW_Push_SPST_NO_Alps_SKRK, symbol Switch:SW_Push
Connections:
- net labels added: PA0, PA1, PA10, PA13, PA8, PA9, PB0, PB1, PB2, PB8, PB9, RESET
- wire segments 142 -> 170
- no-connect marks 25 -> 13
Other:
- moved on the sheet: R7
